File: SIM7600_Breakout.kicad_sch (KiCad schematic)
At the start: 60 parts, among them J1 SIM8060-6-0-14-00-A, J2 2H header, J3 MJ-3502N, J4 30H Header, J5 USB_B_Micro, J6 U.FL-R-SMT-1(01), J7 U.FL-R-SMT-1(01), J8 U.FL-R-SMT-1(01), Q1 MMBT3904L_RFG, U1 NVT2008PW_118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

Commit message: Documentation updates + pics
Parts:
- J2: value 2H header -> 2W Header
- J4: value 30H Header -> 30W Header
Changed lines of the file:
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@@
       (effects (font (size 1.27 1.27)) (justify right))
     )
-    (property "Value" "2H header" (id 1) (at 246.634 115.062 90)
+    (property "Value" "2W Header" (id 1) (at 246.634 115.062 90)
       (effects (font (size 1.27 1.27)) (justify right))
     )
@@
       (effects (font (size 1.27 1.27)) (justify right))
     )
-    (property "Value" "30H Header" (id 1) (at 274.32 53.848 90)
+    (property "Value" "30W Header" (id 1) (at 274.32 53.848 90)
       (effects (font (size 1.27 1.27)) (justify right))
     )
@@
     )
     (path "/854eda8f-d37e-49df-aa08-450e402f5b4c"
-      (reference "J2") (unit 1) (value "2H header") (footprint "Connector_PinHeader_2.54mm:PinHeader_1x02_P2.54mm_Vertical")
+      (reference "J2") (unit 1) (value "2W Header") (footprint "Connector_PinHeader_2.54mm:PinHeader_1x02_P2.54mm_Vertical")
     )
     (path "/309204ef-7373-426d-8821-f8b478a9ccbb"
@@
     )
     (path "/8a6937b9-f64b-4379-a3aa-862c0016b2c6"
-      (reference "J4") (unit 1) (value "30H Header") (footprint "Connector_PinHeader_2.54mm:PinHeader_1x30_P2.54mm_Vertical")
+      (reference "J4") (unit 1) (value "30W Header") (footprint "Connector_PinHeader_2.54mm:PinHeader_1x30_P2.54mm_Vertical")
     )
     (path "/778c53f9-d110-4358-bf3e-2d1ecc97e325"

Commit message: Minor fixes
Parts:
- renumbered D4 to D3, D3 to D4
Changed lines of the file:
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@@
   (symbol (lib_id "ESD9L5.0ST5G:ESD9L5.0ST5G") (at 208.788 76.327 90) (unit 1)
     (in_bom yes) (on_board yes)
-    (property "Reference" "D4" (id 0) (at 210.058 78.867 0)
+    (property "Reference" "D3" (id 0) (at 210.058 78.867 0)
       (effects (font (size 1.27 1.27)) (justify right))
     )
@@
   (symbol (lib_id "ESD9L5.0ST5G:ESD9L5.0ST5G") (at 215.773 76.327 90) (unit 1)
     (in_bom yes) (on_board yes)
-    (property "Reference" "D3" (id 0) (at 217.043 78.867 0)
+    (property "Reference" "D4" (id 0) (at 217.043 78.867 0)
       (effects (font (size 1.27 1.27)) (justify right))
     )
@@
       (reference "D2") (unit 1) (value "R_LED") (footprint "LED_SMD:LED_1206_3216Metric_Pad1.42x1.75mm_HandSolder")
     )
+    (path "/548c3e4a-6797-4003-bf6e-b7e438abf8b4"
+      (reference "D3") (unit 1) (value "ESD9L5.0ST5G") (footprint "sim7600_breakout:DIOM1006X40N")
+    )
     (path "/8928f370-2f24-4aae-b99f-ebcb925524b4"
-      (reference "D3") (unit 1) (value "ESD9L5.0ST5G") (footprint "sim7600_breakout:DIOM1006X40N")
-    )
-    (path "/548c3e4a-6797-4003-bf6e-b7e438abf8b4"
       (reference "D4") (unit 1) (value "ESD9L5.0ST5G") (footprint "sim7600_breakout:DIOM1006X40N")
     )
